File: 250407_sheet2.sch (KiCad schematic (older format))
At the start: 90 parts, among them CN5 AV_CONN, CN6 EXPANSION_PORT, M1 MODULATOR_LONGBOARD, Q8 2SC1815, U10 4164-2, U11 4164-2, U12 4164-2, U13 74LS257, U14 74LS258, U15 74LS139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

Commit message: Update schematics version and readme
Parts:
- CN5: symbol KU-schematics-library:AV_CONN -> 250407_-rescue:AV_CONN-KU-schematics-library
- CN6: symbol KU-schematics-library:EXPANSION_PORT -> 250407_-rescue:EXPANSION_PORT-KU-schematics-library
- FB10, FB11, FB12, FB13, FB14, FB15, FB22, FB4: symbol KU-schematics-library:FERRITE_BEAD -> 250407_-rescue:FERRITE_BEAD-KU-schematics-library
- RP1, RP2: symbol KU-schematics-library:R_ARRAY_US_4RES -> 250407_-rescue:R_ARRAY_US_4RES-KU-schematics-library
- U10, U11, U12, U21, U22, U23, U24, U9: symbol KU-schematics-library:4164-2 -> 250407_-rescue:4164-2-KU-schematics-library
- U13: symbol KU-schematics-library:74LS257_U13 -> 250407_-rescue:74LS257_U13-KU-schematics-library
- U14: symbol KU-schematics-library:74LS258 -> 250407_-rescue:74LS258-KU-schematics-library
- U16: symbol KU-schematics-library:4066_U28 -> 250407_-rescue:4066_U28-KU-schematics-library
- U18: symbol KU-schematics-library:SID -> 250407_-rescue:SID-KU-schematics-library
- U19: symbol KU-schematics-library:VIC -> 250407_-rescue:VIC-KU-schematics-library
- U25: symbol KU-schematics-library:74LS257 -> 250407_-rescue:74LS257-KU-schematics-library
- U26: symbol KU-schematics-library:74LS373 -> 250407_-rescue:74LS373-KU-schematics-library
- U27: symbol KU-schematics-library:7408_U27 -> 250407_-rescue:7408_U27-KU-schematics-library
- U3, U4: symbol KU-schematics-library:2364A_ROM -> 250407_-rescue:2364A_ROM-KU-schematics-library
- U5: symbol KU-schematics-library:2332A_ROM -> 250407_-rescue:2332A_ROM-KU-schematics-library
Changed lines of the file:
@@
 $EndDescr
 $Comp
-L KU-schematics-library:R_ARRAY_US_4RES RP1
+L 250407_-rescue:R_ARRAY_US_4RES-KU-schematics-library RP1
 U 1 1 60633A40
 P 3600 1950
@@
 $EndComp
 $Comp
-L KU-schematics-library:R_ARRAY_US_4RES RP1
+L 250407_-rescue:R_ARRAY_US_4RES-KU-schematics-library RP1
 U 2 1 60633A46
 P 3600 2150
@@
 $EndComp
 $Comp
-L KU-schematics-library:R_ARRAY_US_4RES RP1
+L 250407_-rescue:R_ARRAY_US_4RES-KU-schematics-library RP1
 U 3 1 60633A4C
 P 3600 2050
@@
 $EndComp
 $Comp
-L KU-schematics-library:R_ARRAY_US_4RES RP1
+L 250407_-rescue:R_ARRAY_US_4RES-KU-schematics-library RP1
 U 4 1 60633A52
 P 3600 1850
@@
 33
 $Comp
-L KU-schematics-library:74LS257 U25
+L 250407_-rescue:74LS257-KU-schematics-library U25
 U 1 1 60633A5A
 P 2350 3800
@@
 33
 $Comp
-L KU-schematics-library:R_ARRAY_US_4RES RP2
+L 250407_-rescue:R_ARRAY_US_4RES-KU-schematics-library RP2
 U 4 1 60633A6E
 P 3600 2450
@@
 $EndComp
 $Comp
-L KU-schematics-library:R_ARRAY_US_4RES RP2
+L 250407_-rescue:R_ARRAY_US_4RES-KU-schematics-library RP2
 U 3 1 60633A74
 P 3600 2350
@@
 $EndComp
 $Comp
-L KU-schematics-library:R_ARRAY_US_4RES RP2
+L 250407_-rescue:R_ARRAY_US_4RES-KU-schematics-library RP2
 U 1 1 60633A7A
 P 3600 2250
@@
 ~CAS~
 $Comp
-L KU-schematics-library:R_ARRAY_US_4RES RP2
+L 250407_-rescue:R_ARRAY_US_4RES-KU-schematics-library RP2
 U 2 1 60633A98
 P 3600 2550
@@
 A0
 $Comp
-L KU-schematics-library:4164-2 U12
+L 250407_-rescue:4164-2-KU-schematics-library U12
 U 1 1 60633ACE
 P 4150 2400
@@
 	2300 1250 2300 1800
 $Comp
-L KU-schematics-library:74LS257_U13 U13
+L 250407_-rescue:74LS257_U13-KU-schematics-library U13
 U 1 1 60633B47
 P 2350 2350
@@
 ~CASRAM~'
 $Comp
-L KU-schematics-library:7408_U27 U27
+L 250407_-rescue:7408_U27-KU-schematics-library U27
 U 2 1 60633B50
 P 1400 6300
@@
 R\~W~
 $Comp
-L KU-schematics-library:2364A_ROM U3
+L 250407_-rescue:2364A_ROM-KU-schematics-library U3
 U 1 1 60633B6E
 P 4150 6000
@@
 BFFF)
 $Comp
-L KU-schematics-library:2364A_ROM U4
+L 250407_-rescue:2364A_ROM-KU-schematics-library U4
 U 1 1 60633B78
 P 5500 6000
@@
 A0
 $Comp
-L KU-schematics-library:2332A_ROM U5
+L 250407_-rescue:2332A_ROM-KU-schematics-library U5
 U 1 1 60633C41
 P 6850 6000
@@
 R\~W~
 $Comp
-L KU-schematics-library:EXPANSION_PORT CN6
+L 250407_-rescue:EXPANSION_PORT-KU-schematics-library CN6
 U 1 1 60633CA9
 P 3350 10500
@@
 	2600 10050 2600 10300
 $Comp
-L KU-schematics-library:FERRITE_BEAD FB?
+L 250407_-rescue:FERRITE_BEAD-KU-schematics-library FB?
 U 1 1 60633CED
 P 1900 9600
@@
 	2900 1050 1600 1050
 $Comp
-L KU-schematics-library:74LS258 U14
+L 250407_-rescue:74LS258-KU-schematics-library U14
 U 1 1 60633EA7
 P 9800 1400
@@
 ~VA14~
 $Comp
-L KU-schematics-library:4066_U28 U16
+L 250407_-rescue:4066_U28-KU-schematics-library U16
 U 1 1 60633ED5
 P 9900 3350
@@
 	9150 1250 9450 1250
 $Comp
-L KU-schematics-library:VIC U?
+L 250407_-rescue:VIC-KU-schematics-library U?
 U 1 1 60633EE5
 P 11850 3600
@@
 $EndComp
 $Comp
-L KU-schematics-library:74LS373 U26
+L 250407_-rescue:74LS373-KU-schematics-library U26
 U 1 1 60633F0C
 P 8400 6200
@@
 AEC
 $Comp
-L KU-schematics-library:4164-2 U24
+L 250407_-rescue:4164-2-KU-schematics-library U24
 U 1 1 60633F47
 P 4650 2400
@@
 ~RAS~
 $Comp
-L KU-schematics-library:4164-2 U11
+L 250407_-rescue:4164-2-KU-schematics-library U11
 U 1 1 60633F63
 P 5150 2400
@@
 ~RAS~
 $Comp
-L KU-schematics-library:4164-2 U23
+L 250407_-rescue:4164-2-KU-schematics-library U23
 U 1 1 60633F7F
 P 5650 2400
@@
 ~RAS~
 $Comp
-L KU-schematics-library:4164-2 U10
+L 250407_-rescue:4164-2-KU-schematics-library U10
 U 1 1 60633F9B
 P 6150 2400
@@
 ~RAS~
 $Comp
-L KU-schematics-library:4164-2 U22
+L 250407_-rescue:4164-2-KU-schematics-library U22
 U 1 1 60633FB7
 P 6650 2400
@@
 ~RAS~
 $Comp
-L KU-schematics-library:4164-2 U21
+L 250407_-rescue:4164-2-KU-schematics-library U21
 U 1 1 60633FE9
 P 7650 2400
@@
 	3900 3250 3900 4500
 $Comp
-L KU-schematics-library:4164-2 U9
+L 250407_-rescue:4164-2-KU-schematics-library U9
 U 1 1 60634009
 P 7150 2400
@@
 $EndComp
 $Comp
-L KU-schematics-library:7408_U27 U27
+L 250407_-rescue:7408_U27-KU-schematics-library U27
 U 3 1 60634169
 P 10250 7500
@@
 	12450 1650 12800 1650
 $Comp
-L KU-schematics-library:FERRITE_BEAD FB?
+L 250407_-rescue:FERRITE_BEAD-KU-schematics-library FB?
 U 1 1 60634221
 P 13100 1650
@@
 $EndComp
 $Comp
-L KU-schematics-library:FERRITE_BEAD FB?
+L 250407_-rescue:FERRITE_BEAD-KU-schematics-library FB?
 U 1 1 60634230
 P 12700 2150
@@
 	13500 3100 13300 2700
 $Comp
-L KU-schematics-library:FERRITE_BEAD FB?
+L 250407_-rescue:FERRITE_BEAD-KU-schematics-library FB?
 U 1 1 60634280
 P 12550 3300
@@
 $EndComp
 $Comp
-L KU-schematics-library:FERRITE_BEAD FB?
+L 250407_-rescue:FERRITE_BEAD-KU-schematics-library FB?
 U 1 1 60634286
 P 12550 3200
@@
 $EndComp
 $Comp
-L KU-schematics-library:FERRITE_BEAD FB?
+L 250407_-rescue:FERRITE_BEAD-KU-schematics-library FB?
 U 1 1 60634302
 P 14150 5600
@@
 $EndComp
 $Comp
-L KU-schematics-library:FERRITE_BEAD FB?
+L 250407_-rescue:FERRITE_BEAD-KU-schematics-library FB?
 U 1 1 60634341
 P 14150 5000
@@
 $EndComp
 $Comp
-L KU-schematics-library:FERRITE_BEAD FB?
+L 250407_-rescue:FERRITE_BEAD-KU-schematics-library FB?
 U 1 1 6063437A
 P 14150 4600
@@
 $EndComp
 $Comp
-L KU-schematics-library:SID U18
+L 250407_-rescue:SID-KU-schematics-library U18
 U 1 1 60634390
 P 13350 5600
@@
 	12650 5900 12850 5900
 $Comp
-L KU-schematics-library:AV_CONN CN5
+L 250407_-rescue:AV_CONN-KU-schematics-library CN5
 U 1 1 606343A4
 P 15650 3650
@@
 	12750 3300 13500 3300
 $Comp
-L KU-schematics-library:7408_U27 U27
+L 250407_-rescue:7408_U27-KU-schematics-library U27
 U 4 1 60633B5A
 P 1400 8300
