File: 250407_.sch (KiCad schematic (older format))
At the start: 132 parts, among them CN1 KEYBOARD_20PIN_MALE, CN10 LED_CONNECTOR, CN2 USER_PORT_CON, CN3 CASSETTE_PORT_CON, CN4 SERIAL_BUS_CON, CN7 POWER_CON, CN8 CONTROL_PORT, CN9 CONTROL_PORT, Q1 2SC1815, Q2 2SC1815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

Commit message: TP29B #2
Parts:
- Q3: value TP298/2SD880 -> TP29B/2SD880
Changed lines of the file:
@@
 P 9150 1650
 F 0 "Q3" H 9341 1696 50  0000 L CNN
-F 1 "TP298/2SD880" H 9341 1605 50  0000 L CNN
+F 1 "TP29B/2SD880" H 9341 1605 50  0000 L CNN
 F 2 "KU-14194HB-RevB-KiCad:TO-220-3_Horizontal_TabDown_250407" H 9400 1575 50  0001 L CIN
 F 3 "https://www.centralsemi.com/get_document.php?cmp=1&mergetype=pd&mergepath=pd&pdf_id=tip41.PDF" H 9150 1650 50  0001 L CNN

Commit message: Update schematics version and readme
Parts:
- CN2: symbol KU-schematics-library:USER_PORT_CON -> 250407_-rescue:USER_PORT_CON-KU-schematics-library
- CN7: symbol KU-schematics-library:POWER_CON -> 250407_-rescue:POWER_CON-KU-schematics-library
- CN8, CN9: symbol KU-schematics-library:CONTROL_PORT -> 250407_-rescue:CONTROL_PORT-KU-schematics-library
- FB18: symbol KU-schematics-library:FERRITE_BEAD -> 250407_-rescue:FERRITE_BEAD-KU-schematics-library
- L4: symbol KU-schematics-library:CHOKE -> 250407_-rescue:CHOKE-KU-schematics-library
- U27: symbol KU-schematics-library:7408_U27 -> 250407_-rescue:7408_U27-KU-schematics-library
- U28: symbol KU-schematics-library:4066_U28 -> 250407_-rescue:4066_U28-KU-schematics-library
- U29: symbol KU-schematics-library:74LS74 -> 250407_-rescue:74LS74-KU-schematics-library
- U30: symbol KU-schematics-library:74LS193 -> 250407_-rescue:74LS193-KU-schematics-library
- U31: symbol KU-schematics-library:74LS629N -> 250407_-rescue:74LS629N-KU-schematics-library
- U32: symbol KU-schematics-library:MC4044 -> 250407_-rescue:MC4044-KU-schematics-library
- U7: symbol KU-schematics-library:6510_MPU -> 250407_-rescue:6510_MPU-KU-schematics-library
Changed lines of the file:
@@
 Sheet 1 2
 Title "C64 250407 PCB Replica"
-Date "2021-06-19"
-Rev "1.1"
+Date "2022-08-18"
+Rev "1.2"
 Comp ""
 Comment1 "by BWACK"
 Comment2 "with help from Der Alte Bastler"
-Comment3 ""
+Comment3 "Schematics V1.2 for Board V1.1"
 Comment4 ""
 $EndDescr
@@
 	1550 1500 1550 1600
 $Comp
-L KU-schematics-library:FERRITE_BEAD FB18
+L 250407_-rescue:FERRITE_BEAD-KU-schematics-library FB18
 U 1 1 605D0086
 P 1800 2700
@@
 $EndComp
 $Comp
-L KU-schematics-library:USER_PORT_CON CN2
+L 250407_-rescue:USER_PORT_CON-KU-schematics-library CN2
 U 1 1 605D0092
 P 1500 9100
@@
 (MALE DB9)
 $Comp
-L KU-schematics-library:CONTROL_PORT CN8
+L 250407_-rescue:CONTROL_PORT-KU-schematics-library CN8
 U 1 1 605D013F
 P 1500 3300
@@
 $EndComp
 $Comp
-L KU-schematics-library:CONTROL_PORT CN9
+L 250407_-rescue:CONTROL_PORT-KU-schematics-library CN9
 U 1 1 605D0145
 P 1500 4400
@@
 Connection ~ 2250 1650
 $Comp
-L KU-schematics-library:4066_U28 U28
+L 250407_-rescue:4066_U28-KU-schematics-library U28
 U 1 1 605D023D
 P 2300 2000
@@
 	11750 7650 11700 7650
 $Comp
-L KU-schematics-library:6510_MPU U7
+L 250407_-rescue:6510_MPU-KU-schematics-library U7
 U 1 1 605D02F0
 P 5950 3050
@@
 9VAC~~
 $Comp
-L KU-schematics-library:7408_U27 U27
+L 250407_-rescue:7408_U27-KU-schematics-library U27
 U 1 1 605D0438
 P 6700 10700
@@
 $EndComp
 $Comp
-L KU-schematics-library:CHOKE L4
+L 250407_-rescue:CHOKE-KU-schematics-library L4
 U 1 1 605D06B2
 P 9900 9950
@@
 (7PIN MALE DIN)
 $Comp
-L KU-schematics-library:POWER_CON CN7
+L 250407_-rescue:POWER_CON-KU-schematics-library CN7
 U 1 1 605D06C8
 P 10550 10750
@@
 Connection ~ 10800 10650
 $Comp
-L KU-schematics-library:74LS629N U31
+L 250407_-rescue:74LS629N-KU-schematics-library U31
 U 1 1 605D083A
 P 9500 6700
@@
 	10100 4250 10100 4300
 $Comp
-L KU-schematics-library:74LS629N U31
+L 250407_-rescue:74LS629N-KU-schematics-library U31
 U 2 1 605D08D0
 P 10100 3950
@@
 $EndComp
 $Comp
-L KU-schematics-library:74LS74 U29
+L 250407_-rescue:74LS74-KU-schematics-library U29
 U 1 1 605D0930
 P 11850 3500
@@
 $EndComp
 $Comp
-L KU-schematics-library:74LS74 U29
+L 250407_-rescue:74LS74-KU-schematics-library U29
 U 2 1 605D0936
 P 12700 5050
@@
 	10150 5900 15250 5900
 $Comp
-L KU-schematics-library:MC4044 U32
+L 250407_-rescue:MC4044-KU-schematics-library U32
 U 1 1 605D09EE
 P 13350 5000
@@
 $EndComp
 $Comp
-L KU-schematics-library:MC4044 U32
+L 250407_-rescue:MC4044-KU-schematics-library U32
 U 2 1 605D09F4
 P 13750 5000
@@
 $EndComp
 $Comp
-L KU-schematics-library:MC4044 U32
+L 250407_-rescue:MC4044-KU-schematics-library U32
 U 3 1 605D09FA
 P 14950 5200
@@
 F_DIV
 $Comp
-L KU-schematics-library:74LS193 U30
+L 250407_-rescue:74LS193-KU-schematics-library U30
 U 1 1 605D0A03
 P 11250 4800

Commit message: replaced CR5, CR6, F1 and CN10 with symbols closer to original schematics
Parts:
- CN10: symbol Connector_Generic:Conn_01x03 -> KU-schematics-library:LED_CONN
- CN2: symbol 250407_-rescue:USER_PORT_CON-KU-schematics-library -> KU-schematics-library:USER_PORT_CON
- CN7: symbol 250407_-rescue:POWER_CON-KU-schematics-library -> KU-schematics-library:POWER_CON
- CN8, CN9: symbol 250407_-rescue:CONTROL_PORT-KU-schematics-library -> KU-schematics-library:CONTROL_PORT
- CR5, CR6: symbol Diode:1N4001 -> Device:D_Small_ALT
- E1: symbol 250407_-rescue:JUMPER_WIRE-KU-schematics-library -> KU-schematics-library:JUMPER_WIRE
- E2: symbol 250407_-rescue:JUMPER_WIRE_DASHED-KU-schematics-library -> KU-schematics-library:JUMPER_WIRE_DASHED
- F1: symbol Device:Fuse -> KU-schematics-library:Fuse_ALT
- FB18: symbol 250407_-rescue:FERRITE_BEAD-KU-schematics-library -> KU-schematics-library:FERRITE_BEAD
- L4: symbol 250407_-rescue:CHOKE-KU-schematics-library -> KU-schematics-library:CHOKE
- SW1: symbol 250407_-rescue:POWER_SWITCH-KU-schematics-library -> KU-schematics-library:POWER_SWITCH
- U27: symbol 250407_-rescue:7408_U27-KU-schematics-library -> KU-schematics-library:7408_U27
- U28: symbol 250407_-rescue:4066_U28-KU-schematics-library -> KU-schematics-library:4066_U28
- U29: symbol 250407_-rescue:74LS74-KU-schematics-library -> KU-schematics-library:74LS74
- U30: symbol 250407_-rescue:74LS193-KU-schematics-library -> KU-schematics-library:74LS193
- U31: symbol 250407_-rescue:74LS629N-KU-schematics-library -> KU-schematics-library:74LS629N
- U32: symbol 250407_-rescue:MC4044-KU-schematics-library -> KU-schematics-library:MC4044
- U7: symbol 250407_-rescue:6510_MPU-KU-schematics-library -> KU-schematics-library:6510_MPU
Connections:
- net Earth: now also SW1.pe; no longer SW1.~ (pe)
